Commit message: Changed the IMU offset according to Michele values

File: robots/hyq.urdf.xacro (robot description, xacro)
@@ -73,5 +73,5 @@
 		update_rate="100.0"
 		stdev="0.00017">
-		<origin xyz="0.3 0 0.095" rpy="0 ${-PI} 0"/>
+		<origin xyz="0.4825 0.006 0.0905" rpy="0 ${-PI} 0"/>
 	</xacro:microstrain_3dmgx325_imu>
 	<!-- Velodyne -->
